File: electronics/carrier/carrier.kicad_sch (KiCad schematic)
At the start: 65 parts, among them J1 PJ-063AH, J2 USB-C power in, J3 S3 USB (P4 link, flashing), J4 5V to P4, J5 HUB75, J6 LED panel 5V, J7 INMP441, J8 P4 UART (future), SW1 Reset, SW2 Boot, U1 ESP32-S3-WROOM-1-N16R8, U2 CH224A, U3 TPS568215, U4 USBLC6-2SC6, U5 AP2112K-3.3, U6 74AHCT245, U7 74AHCT245

Commit message: Route the carrier board
Add route_board.py: locked high-current and fine-pitch copper, Freerouting
for the rest, ground pours and stitching vias, then KiCad's own check for
anything left unconnected. The board passes DRC with no errors, nothing
unconnected and exact schematic parity.

- Remove the solder jumpers: F1 alone selects the barrel input, and the
  USB-C buck output feeds +5V directly.
- Name stacked unconnected pins as KiCad does, so the S3 socket's paired
  VBUS pads share one net.
- Rotate U3 so its switch node runs straight to L1; move the MODE/EN
  dividers and the boot capacitor to suit. Swap R3/R4 to match their CC pins.
- Hide chip passive references on the silkscreen; allow ref positions in
  board.json; allow one thermal spoke on through-hole pads (.kicad_dru).

Co-Authored-By: Claude Opus 5.5 <noreply@anthropic.com>
Parts:
- removed JP1: Barrel input, Jumper:SolderJumper-2_P1.3mm_Bridged_RoundedPad1.0x1.5mm, symbol Jumper:SolderJumper_2_Bridged
- removed JP2: USB-C input, Jumper:SolderJumper-2_P1.3mm_Open_RoundedPad1.0x1.5mm, symbol Jumper:SolderJumper_2_Open
- F1: Note (none) -> Also selects the barrel input: fit F1 or the USB-C power se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
- J3: Note VBUS from the P4 is not connected to the board's 5 V rail. -> VBUS pins unconnected: the P4's 5 V never feeds the board's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
Connections:
- net BUCK_OUT is gone; now on net +5V: C12.1, C19.1, C20.1, C21.1, C22.1, C23.1, L1.2, R11.1
- net VIN_FUSED is gone; now on net +5V: F1.2
- net S3_VBUS: no longer names the net of J3.A4 (VBUS), J3.A9 (VBUS), J3.B4 (VBUS), J3.B9 (VBUS)
- no-connect marks 37 -> 38
Other:
- moved on the sheet: C1, C2, C3, D1

Commit message: Use a latching JST GH socket for the microphone
The PH socket held by friction only. Hand-draw the R13 sense link the
autorouter sometimes misses, and drop stitching vias that land on
isolated pour islands.

Co-Authored-By: Claude Opus 5.5 <noreply@anthropic.com>
Parts:
- J7: footprint Connector_JST:JST_PH_B6B-PH-K_1x06_P2.00mm_Vertical -> Connector_JST:JST_GH_BM06B-GHS-TBT_1x06-1MP_P1.25mm_Vertical
Changed lines of the file:
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@@
 			)
 		)
-		(property "Footprint" "Connector_JST:JST_PH_B6B-PH-K_1x06_P2.00mm_Vertical"
+		(property "Footprint" "Connector_JST:JST_GH_BM06B-GHS-TBT_1x06-1MP_P1.25mm_Vertical"
 			(at 632.46 60.96 0)
 			(effects
